File: Eagle/Becca Sap Flow Power Board MOD.brd (EAGLE design)
At the start: 49 x 68.3 mm, 42 parts, among them J1 1935161, J2 1935200, U1 V_REG_317SMD, U2 V_REG_317SMD, U3 V_REG_317SMD

Commit message: Progress
Parts:
- removed FID2: FIDUCIAL_1MM, microbuilder:FIDUCIAL_1MM
- removed U$11: MOUNTINGHOLE2.5, microbuilder:MOUNTINGHOLE_2.5_PLATED
- F1, F2, F3, F4, F5, F6: device Fuse Holder:01020071Z -> Becca-Sap-Flow-LORA:01020071Z
- J1: device Dual Mono Amp Library:1935161 -> Becca-Sap-Flow-LORA:1935161
- J2: device 1935200:1935200 -> Becca-Sap-Flow-LORA:1935200
- JP1, JP2, JP3: device 6P1_EVB:HDR2X1 -> Becca-Sap-Flow-LORA:HDR2X1
- U$1, U$2, U$3, U$4, U$5: value MOUNTINGHOLE2.5 -> MOUNT-HOLE3.0; device microbuilder:MOUNTINGHOLE_2.5_PLATED -> Becca-Sap-Flow-LORA:3,0
- moved D4 223.5 mm to (37.1, 30.6), turned to 90 degrees
- moved C2 208.2 mm to (43.4, 25.1), turned to 180 degrees
- moved U3 186.9 mm to (43.4, 16.8), turned to 90 degrees
- moved D3 182.5 mm to (31.8, 30.6), turned to 90 degrees
- moved C1 169.1 mm to (26.0, 30.6), turned to 270 degrees
- moved U2 154.7 mm to (18.8, 30.6)
- moved D2 147.1 mm to (40.0, 38.1), flipped to the bottom, turned to 135 degrees
- moved D1 108.1 mm to (29.7, 34.9), flipped to the bottom, turned to 180 degrees
- moved U1 29.7 mm to (5.65, 16.8), turned to 90 degrees
- moved D5 22.3 mm to (17.5, 34.9), flipped to the bottom, turned to 180 degrees
- moved C7 17.9 mm to (5.65, 25.1), turned to 0 degrees
- moved D6 16.9 mm to (11.9, 30.6), turned to 90 degrees
- moved R10 5.88 mm to (7.19, 27.0), flipped to the bottom, turned to 0 degrees
- moved R4 5.88 mm to (41.8, 27.0), flipped to the bottom, turned to 180 degrees
- moved F5 4.08 mm to (41.4, 60.0)
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Routing:
- net N$1: track 0.00 -> 38.5 mm
- net VCC3: track 0.00 -> 24.0 mm, vias 0 -> 1
- net N$12: track 3.73 -> 23.3 mm, vias 0 -> 2
- net N$11: track 3.73 -> 22.5 mm, vias 0 -> 2
- net VCC2: track 0.00 -> 18.7 mm, vias 0 -> 1
- net N$7: track 0.00 -> 18.6 mm, vias 0 -> 1
- net N$14: track 0.00 -> 18.5 mm
- net N$13: track 0.00 -> 16.0 mm, vias 0 -> 1
- net OUTPUT1: track 19.4 -> 34.8 mm
- net OUTPUT3: track 19.4 -> 34.8 mm
- net N$2: track 3.73 -> 17.7 mm, vias 0 -> 2
- net N$4: track 0.00 -> 7.26 mm
- net N$9: track 0.00 -> 7.06 mm
- net N$3: track 0.00 -> 6.95 mm
- net N$6: track 0.00 -> 6.37 mm
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
Commit message: Finished boards, generated gerbers and BOM
Parts:
- C1, C2, C7: device rcl:PANASONIC_C -> Becca-Sap-Flow-LORA:CAPAE830X1080N
- D1, D2, D3, D4, D5, D6: device S1A:DIOM5027X250N -> Becca-Sap-Flow-LORA:DIOM5027X250N
- F1, F2, F3, F4, F5, F6: value 01020071Z -> 01110501Z; device Becca-Sap-Flow-LORA:01020071Z -> Becca-Sap-Flow-LORA:01110501Z
- R1, R10, R12, R13, R2, R3, R4, R5, R6: device rcl:R1210 -> Becca-Sap-Flow-LORA:R1210
- U1, U2, U3: value V_REG_317SMD -> LM317MBSTT3G; device SparkFun-IC-Power:SOT223 -> Becca-Sap-Flow-LORA:SOT230P700X175-4N
- VR1, VR2, VR3: device 3296W-1-102RLF:3296W1102RLF -> Becca-Sap-Flow-LORA:3296W1102RLF
- moved D3 9.81 mm to (22.7, 34.4), flipped to the bottom, turned to 270 degrees
- moved D4 4.60 mm to (34.5, 34.4), flipped to the bottom, turned to 270 degrees
- moved D6 3.92 mm to (10.9, 34.4), flipped to the bottom, turned to 270 degrees
- moved F6 3.00 mm to (38.9, 45.0), turned to 90 degrees
- moved C1 2.50 mm to (28.5, 30.6), turned to 0 degrees
- moved F1 2.50 mm to (20.0, 55.9), turned to 270 degrees
- moved F2 2.50 mm to (15.0, 40.9), turned to 90 degrees
- moved F3 2.50 mm to (32.2, 55.9), turned to 270 degrees
- moved F4 2.50 mm to (27.2, 40.9), turned to 90 degrees
- moved F5 2.50 mm to (43.9, 60.0), turned to 270 degrees
- moved VR1 2.50 mm to (17.0, 21.1)
- moved VR3 2.50 mm to (32.0, 21.1)
- moved D2 1.84 mm to (40.9, 39.7)
- moved U1 1.79 mm to (5.65, 15.0), turned to 270 degrees
- moved U3 1.79 mm to (43.4, 15.0), turned to 270 degrees
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Connections:
- removed net GND: C1.-, C2.-, C7.-, J1.2, J2.1, J2.3, J2.5
- new net DGND: C1.2, C2.2, C7.2, J1.2, J2.1, J2.3, J2.5
- net N$3: now also F1.2
- net N$4: now also F3.2
- net N$5: now also F2.1
- net N$6: now also F4.1
- net N$8: now also F5.2
- net N$9: now also F6.1
- net VCC1: now also C7.1; no longer C7.+
- net VCC2: now also C1.1; no longer C1.+
- net VCC3: now also C2.1; no longer C2.+
Routing:
- net OUTPUT3: track 34.8 -> 44.8 mm
- net VCC1: track 19.5 -> 28.4 mm
- net OUTPUT1: track 34.8 -> 43.0 mm
- net N$12: track 23.3 -> 15.1 mm, vias 2 -> 1
- net N$8: track 5.00 -> 11.2 mm
- net N$4: track 7.26 -> 12.8 mm
- net N$11: track 22.5 -> 17.2 mm, vias 2 -> 1
- net N$3: track 6.95 -> 11.9 mm
- net N$5: track 6.37 -> 9.85 mm
- net N$7: track 18.6 -> 15.2 mm
- net N$2: track 17.7 -> 21.1 mm, vias 2 -> 1
- net N$6: track 6.37 -> 9.69 mm
- net OUTPUT2: track 37.4 -> 34.2 mm
- net N$16: track 6.16 -> 8.66 mm
- net N$15: track 6.16 -> 8.66 mm
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- added copper zone on layer 1, net DGND
- added copper zone on layer 16, net DGND
- removed copper zone on layer 1, net GND
- removed copper zone on layer 16, net GND
Other:
- board text added: "+"
- board text added: "1"
- board text added: "1+"
- board text added: "1-"
- board text added: "1A Fuse"
- board text added: "2"
- board text added: "2+"
- board text added: "2-"
- board text added: "3"
- board text added: "3+"
- board text added: "3-"
- board text added: "Sapflow V1.0"
