File: Eagle/Becca Sap Flow Power Board v1_3.brd (EAGLE design)
At the start: 49 x 68.3 mm, 45 parts, among them J1 1935161, J2 1935200, U1 LM317MBSTT3G, U2 LM317MBSTT3G, U3 LM317MBSTT3G

Commit message: More new board progress
Parts:
- added FB1, FB2, FB3: ILHB0805ER600V, Becca-Sap-Flow-LORA:BEADC2012X110N
- C4: value (none) -> 450p
- C5: value (none) -> UWT1E221MNL1GS; device rcl:E2,5-6 -> Becca-Sap-Flow-LORA:CAPAE830X1080N
- L1: value (none) -> IHLP4040EDER750M5A; device rcl:L5650M -> Becca-Sap-Flow-LORA:INDPM115103X540N
- R7: value (none) -> 143m
- R9: value (none) -> 24.9k
- moved C5 40.4 mm to (-31.1, -51.2)
Connections:
- net DGND: now also C5.2; no longer C5.-
- net N$20: now also C5.1; no longer C5.+
