File: Eagle/Becca Sap Flow Power Board v1_3.sch (EAGLE design)
At the start: 45 parts, among them J1 1935161, J2 1935200, U1 LM317MBSTT3G, U2 LM317MBSTT3G, U3 LM317MBSTT3G

Commit message: More new board progress
Parts:
- added FB1, FB2, FB3: ILHB0805ER600V, Becca-Sap-Flow-LORA:ILHB0805ER600V
- C4: value (none) -> 450p
- C5: value (none) -> UWT1E221MNL1GS; device rcl:CPOL-USE2.5-6 -> Becca-Sap-Flow-LORA:UWT1E221MNL1GS
- L1: value (none) -> IHLP4040EDER750M5A; device rcl:L-USL5650M -> Becca-Sap-Flow-LORA:IHLP4040EDER750M5A
- R7: value (none) -> 143m
- R9: value (none) -> 24.9k
Connections:
- net DGND: now also C5.2; no longer C5.-
- net N$20: now also C5.1; no longer C5.+
Other:
- moved on the sheet: C6, F1, F2, F3, JP1, JP2, JP3, L2
